File: 82S1xx_W27C512_Adapter.kicad_pcb (KiCad board)
At the start: 2 copper layers, 20.5 x 37.7 mm, 4 parts, among them J1 82S129, U1 W27C512

Commit message: Add license, ready for V1 and go-public
Parts:
- added V0: LICENSE, 82S1xx_W27C512_Adapter:cc_by_nc_sa, B.Cu at (154.7, 102.7)
Routing:
- net /a0: track 10.2 -> 6.65 mm
Other:
- board text added: "github.com/ SukkoPera/ OldPromAdapter"
